Commit message: Refine arm collision envelopes and add independent CAD visibility

File: model/viscous_arm.urdf (robot description, URDF)
Before this commit: robot viscous_arm_dry_cad_v1, 10 links, 9 joints
Links:
- link base_link: geometry collision mesh filename=meshes/collision_000.stl; collision mesh filename=meshes/collision_002.stl
- link forearm_link: geometry collision mesh filename=meshes/collision_forearm_shell_00.stl; collision mesh filename=meshes/collision_forearm_shell_01.stl
- link gripper_left: geometry collision mesh filename=meshes/collision_032.stl; collision mesh filename=meshes/collision_043_00.stl
- link gripper_right: geometry collision mesh filename=meshes/collision_039.stl; collision mesh filename=meshes/collision_042_00.stl
- link upper_arm_link: geometry collision mesh filename=meshes/collision_upper_arm_shell_00.stl; collision mesh filename=meshes/collision_upper_arm_shell_01.stl
- link wrist_pitch_link: geometry collision mesh filename=meshes/collision_053.stl; collision mesh filename=meshes/collision_054_00.stl
- link wrist_roll_link: geometry collision mesh filename=meshes/collision_020.stl; collision mesh filename=meshes/collision_024_00.stl
- link wrist_yaw_link: geometry collision mesh filename=meshes/collision_049.stl; collision mesh filename=meshes/collision_050_00.stl
- link yaw_link: geometry collision mesh filename=meshes/collision_003_00.stl; collision mesh filename=meshes/collision_003_01.stl
